File: Hardware/Blender/v1_20230918/Design Folder/_HW_Blender/_HW_Blender.kicad_sch (KiCad schematic)
At the start: 0 parts

Commit message: Improving the file structure and documentation
Other:
- added sheet PWR SEQUENCE ([12] - PWR SEQUENCE.kicad_sch)
- added sheet REVISION HISTORY ([13] - REVISION HISTORY.kicad_sch)
- note added: "${COMMENT2}"
- note added: "1- Go to View -> Pge Preview Setting 2- Set Parameters based on the following Info COMMENT 1: Project Version COMMENT 2: Document Status COMMENT 3: Doc. Approval Eng. COMMENT 4: BOM Ref. DOC. COMMENT 5: PCB Ref. DOC. COMMENT 6: GBR Ref. DOC. COMMENT 7: ASM Ref. DOC. COMMENT 8: Variant Name COMMENT 9: Revision Description"
- note added: "1.3" OLED DRIVER"
- note added: "21"
- note added: "22"
- note added: "23"
- note added: "24"
- note added: "25"
- note added: "26"
- note added: "27"
- note added: "28"
- note added: "29"
- note added: "30"
- note added: "3D Preview BOTTOM"
- note added: "3D Preview TOP"
- note added: "BUFFERED VGA INPUT"
- note added: "Board Statistics Stackup Info"
- note added: "ISOLATED DMX"
- note added: "ISOLATED WS28xx DRIVER"
- note added: "MICROCONTROLLER"
- note added: "POWER SUPPLY"
- note added: "SHOULD BE ADDED AFTER RELEASE"
- note added: "SPEAKER DRIVER"
- note added: "TOSLINK RXTX"
- note removed: "1- Go to View -> Pge Preview Setting 2- Set Parameters based on the following Info COMMENT 1: Project Version COMMENT 2: Document Version COMMENT 3: Doc. Approval Eng. COMMENT 4: BOM Ref. DOC. COMMENT 5: PCB Ref. DOC. COMMENT 6: GBR Ref. DOC. COMMENT 7: ASM Ref. DOC. COMMENT 8: Variant Name COMMENT 9: Revision Description"
- note removed: "RELEASED"
