File: Hardware/Blender/v1_20230918/Design Folder/_HW_Blender/[03] - MICROCONTROLLER.kicad_sch (KiCad schematic)
At the start: 25 parts, among them J301 RCPT_4POS_1.27MM, U301 STM32F446RCT6TR, X301 16MHz/10ppm

Commit message: More update for hardware part
Parts:
- C301, C304, C306, C310, C312, C314, C316: value 1uF/6V3 -> 1uF_6V3_X5R; symbol _SCHLIB_Blender:CAP_1uF/6V3_C0201 -> _SCHLIB_Blender:CAP_1uF_6V3_X5R_C0201; Manufacturer (none) -> Samsung Electro-Mechanics; PCB CHECk (none) -> PCB (N/A); Part Number CL03A105MQ3CSNH -> (none); Part Number (Manufacturer) (none) -> CL03A105MQ3CSNH; Part Number (Vendor) (none) -> 1276-6441-2-ND; SCH CHECK CHECKED -> SCH (N/A); Vendor (none) -> Digikey
- C302, C303: value 12pF/50V -> 12pF_50V_C0G; symbol _SCHLIB_Blender:CAP_12pF/50V_C0201 -> _SCHLIB_Blender:CAP_12pF_50V_C0G_C0201; Manufacturer (none) -> YAGEO; PCB CHECk (none) -> PCB (N/A); Part Number CC0201JRNPO9BN120 -> (none); Part Number (Manufacturer) (none) -> CC0201JRNPO9BN120; Part Number (Vendor) (none) -> 311-1585-2-ND; SCH CHECK CHECKED -> SCH (N/A); Vendor (none) -> Digikey
- C305, C307, C311, C313, C315, C317: value 100nF/6V3 -> 100nF_6V3_X7R; symbol _SCHLIB_Blender:CAP_100nF/6V3_C0201 -> _SCHLIB_Blender:CAP_100nF_6V3_X7R_C0201; Manufacturer (none) -> YAGEO; PCB CHECk (none) -> PCB (N/A); Part Number CC0201KRX7R5BB104 -> (none); Part Number (Manufacturer) (none) -> CC0201KRX7R5BB104; Part Number (Vendor) (none) -> 13-CC0201KRX7R5BB104TR-ND; SCH CHECK CHECKED -> SCH (N/A); Vendor (none) -> Digikey
- C308, C309: value 2u2F/6V3 -> 2u2F_6V3_X5R; symbol _SCHLIB_Blender:CAP_2u2F/6V3_C0201 -> _SCHLIB_Blender:CAP_2u2F_6V3_X5R_C0201; Manufacturer (none) -> KYOCERA AVX; PCB CHECk (none) -> PCB (N/A); Part Number CM03X5R225M06AH -> (none); Part Number (Manufacturer) (none) -> CM03X5R225M06AH; Part Number (Vendor) (none) -> 478-KGM03CR50J225MHTR-ND; SCH CHECK CHECKED -> SCH (N/A); Vendor (none) -> Digikey
- J301: value RCPT_4POS_1.27MM -> RECEPT_4X1_VERT_1.27MM; symbol _SCHLIB_Blender:CONN_RCPT_4POS_1.27MM_VERT -> _SCHLIB_Blender:CONN_RECEPT_4POS_1ROW_VERT_1.27MM; Manufacturer (none) -> GCT; PCB CHECk (none) -> PCB (N/A); Package (none) -> THD-VERT-2.54MM; Part Number BD080-04-A-0230-L-D -> (none); Part Number (Manufacturer) (none) -> BD080-04-A-0230-L-D; Part Number (Vendor) (none) -> 2073-BD080-04-A-0230-L-D-ND; SCH CHECK CHECKED -> SCH (N/A); Vendor (none) -> Digikey
- LED301: value RED -> RED_2V; symbol _SCHLIB_Blender:LED_RED_0402 -> _SCHLIB_Blender:DIODE_LED_RED_2V_0.02A_624nm_0402; Manufacturer (none) -> Harvatek Corporation; PCB CHECk (none) -> PCB (N/A); Part Number B2841USD-20D001014U1930 -> (none); Part Number (Manufacturer) (none) -> B2841USD-20D001014U1930; Part Number (Vendor) (none) -> 3147-B2841USD-20D001014U1930TR-ND; SCH CHECK CHECKED -> SCH (N/A); VOLTAGE RATED 2V -> (none); Vendor (none) -> Digikey
- R301, R302: value 10KR_1/20W -> 10KR_1/20W_1%; symbol _SCHLIB_Blender:RES_10KR_1/20W-R0201 -> _SCHLIB_Blender:RES_10KR_1/20W_1%_R0201; Manufacturer (none) -> Stackpole Electronics Inc; PCB CHECk (none) -> PCB (N/A); Part Number RMCF0201FT10K0 -> (none); Part Number (Manufacturer) (none) -> RMCF0201FT10K0; Part Number (Vendor) (none) -> RMCF0201FT10K0TR-ND; SCH CHECK CHECKED -> SCH (N/A); Vendor (none) -> Digikey
- R303: value 49R9_1/20W -> 49R9_1/20W_1%; symbol _SCHLIB_Blender:RES_49R9_1/20W-R0201 -> _SCHLIB_Blender:RES_49R9_1/20W_1%_R0201; Manufacturer (none) -> Stackpole Electronics Inc; PCB CHECk (none) -> PCB (N/A); Part Number RMCF0201FT49R9 -> (none); Part Number (Manufacturer) (none) -> RMCF0201FT49R9; Part Number (Vendor) (none) -> RMCF0201FT49R9TR-ND; SCH CHECK CHECKED -> SCH (N/A); Vendor (none) -> Digikey
- R304: value 100R_1/20W -> 100R_1/20W_1%; symbol _SCHLIB_Blender:RES_100R_1/20W-R0201 -> _SCHLIB_Blender:RES_100R_1/20W_1%_R0201; Manufacturer (none) -> Stackpole Electronics Inc; PCB CHECk (none) -> PCB (N/A); Part Number RMCF0201FT100R -> (none); Part Number (Manufacturer) (none) -> RMCF0201FT100R; Part Number (Vendor) (none) -> RMCF0201FT100RTR-ND; SCH CHECK CHECKED -> SCH (N/A); Vendor (none) -> Digikey
- U301: symbol _SCHLIB_Blender:MCU_STM32F446RCT6TR -> _SCHLIB_Blender:IC_MCU_STM32F446RCT6TR_32bit_64-LQFP (10x10); Manufacturer (none) -> STMicroelectronics; PCB CHECk (none) -> PCB (N/A); Package (none) -> 64-LQFP (10x10); Part Number STM32F446RCT6TR -> (none); Part Number (Manufacturer) (none) -> STM32F446RCT6TR; Part Number (Vendor) (none) -> 497-19357-2-ND; SCH CHECK * -> SCH (N/A); Vendor (none) -> Digikey
- X301: value 16MHz/10ppm -> 16MHz_12pF_10ppm; symbol _SCHLIB_Blender:XTAL_ECS-160-12-37B-CTN-TR -> _SCHLIB_Blender:XTAL_ECS-160-12-37B-CTN-TR_16MHz_12pF_4SMD-1206; Manufacturer (none) -> ECS Inc.; PCB CHECk (none) -> PCB (N/A); Part Number ECS-160-12-37B-CTN-TR -> (none); Part Number (Manufacturer) (none) -> ECS-160-12-37B-CTN-TR; Part Number (Vendor) (none) -> XC3061TR-ND; SCH CHECK CHECKED -> SCH (N/A); Vendor (none) -> Digikey
Other:
- moved on the sheet: C301, C302, C303, C304, C306, C308, C310, C311, C312, C313, C314, C315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
