File: Hardware/Blender/v1_20230918/Design Folder/_HW_Blender/[04] - TOSLINK RXTX.kicad_sch (KiCad schematic)
At the start: 12 parts, among them J401 PLR237/T10BK, J402 TOTX1350(F), U401 SN74LVC1G17DBVR, U402 SN74LVC1G17DBVR

Commit message: Improving the file structure and documentation
Other:
- note removed: "UNCHECKED"
- moved on the sheet: C401, C402, C403, C404, J401, J402, R401, R402, R403, R404, U401, U402

Commit message: More update for hardware part
Parts:
- C401: value 680pF_50V -> 680pF_50V_X7R; symbol _SCHLIB_Blender:CAP_680pF_50V_C0402 -> _SCHLIB_Blender:CAP_680pF_50V_X7R_C0402; Manufacturer (none) -> Walsin Technology Corporation; PCB CHECk (none) -> PCB (N/A); Part Number 0402B681K500CT -> (none); Part Number (Manufacturer) (none) -> 0402B681K500CT; Part Number (Vendor) (none) -> 1292-1223-2-ND; SCH CHECK * -> SCH (N/A); Vendor (none) -> Digikey
- C402, C403, C404: value 100nF/6V3 -> 100nF_6V3_X7R; symbol _SCHLIB_Blender:CAP_100nF/6V3_C0201 -> _SCHLIB_Blender:CAP_100nF_6V3_X7R_C0201; Manufacturer (none) -> YAGEO; PCB CHECk (none) -> PCB (N/A); Part Number CC0201KRX7R5BB104 -> (none); Part Number (Manufacturer) (none) -> CC0201KRX7R5BB104; Part Number (Vendor) (none) -> 13-CC0201KRX7R5BB104TR-ND; SCH CHECK CHECKED -> SCH (N/A); Vendor (none) -> Digikey
- J401: symbol _SCHLIB_Blender:CONN_PLR237/T10BK -> _SCHLIB_Blender:CONN_OPT-RECIEVER_PLR237/T10BK_3V~5V_RA; Manufacturer (none) -> Everlight Electronics Co Ltd; PCB CHECk (none) -> PCB (N/A); Package (none) -> THD-RA; Part Number PLR237/T10BK -> (none); Part Number (Manufacturer) (none) -> PLR237/T10BK; Part Number (Vendor) (none) -> 1080-PLR237/T10BK-ND; SCH CHECK * -> SCH (N/A); Vendor (none) -> Digikey
- J402: symbol _SCHLIB_Blender:CONN_TOTX1350(F) -> _SCHLIB_Blender:CONN_OPT-TRASMITTER_TOTX1350(F)_1.8V_0.030A_RA; Manufacturer (none) -> Toshiba Semiconductor and Storage; PCB CHECk (none) -> PCB (N/A); Package (none) -> THD-RA; Part Number TOTX1350(F) -> (none); Part Number (Manufacturer) (none) -> TOTX1350(F); Part Number (Vendor) (none) -> TOTX1350(F)-ND; SCH CHECK * -> SCH (N/A); Vendor (none) -> Digikey
- R401: value 330R_1/16W -> 330R_1/16W_1%; symbol _SCHLIB_Blender:RES_330R_1/16W_R0402 -> _SCHLIB_Blender:RES_330R_1/16W_1%_R0402; Manufacturer (none) -> Walsin Technology Corporation; PCB CHECk (none) -> PCB (N/A); Part Number WR04X3300FTL -> (none); Part Number (Manufacturer) (none) -> WR04X3300FTL; Part Number (Vendor) (none) -> 1292-WR04X3300FTLTR-ND; SCH CHECK * -> SCH (N/A); Vendor  (none) -> Digikey
- R402: value 100R_1/10W -> 100R_1/10W_1%; symbol _SCHLIB_Blender:RES_100R_1/10W_R0402 -> _SCHLIB_Blender:RES_100R_1/10W_1%_R0402; Manufacturer (none) -> Panasonic Electronic Components; PCB CHECk (none) -> PCB (N/A); Part Number ERJ-2RKF1000X -> (none); Part Number (Manufacturer) (none) -> ERJ-2RKF1000X; Part Number (Vendor) (none) -> P100LTR-ND; SCH CHECK * -> SCH (N/A); Vendor (none) -> Digikey
- R403: value 4K7R_1/20W -> 47KR_1/20W_1%; symbol _SCHLIB_Blender:RES_4K7R_1/20W-R0201 -> _SCHLIB_Blender:RES_47KR_1/20W_1%_R0201; Link https://www.digikey.ca/en/products/detail/stackpole-electro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 -> https://www.digikey.ca/en/products/detail/yageo/AC0201FR-07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; Manufacturer (none) -> YAGEO; PCB CHECk (none) -> PCB (N/A); Part Number RMCF0201FT4K70 -> (none); Part Number (Manufacturer) (none) -> AC0201FR-0747KL; Part Number (Vendor) (none) -> YAG3425TR-ND; SCH CHECK CHECKED -> SCH (N/A); Vendor (none) -> Digikey
- R404: value 10KR_1/20W -> 10KR_1/20W_1%; symbol _SCHLIB_Blender:RES_10KR_1/20W-R0201 -> _SCHLIB_Blender:RES_10KR_1/20W_1%_R0201; Manufacturer (none) -> Stackpole Electronics Inc; PCB CHECk (none) -> PCB (N/A); Part Number RMCF0201FT10K0 -> (none); Part Number (Manufacturer) (none) -> RMCF0201FT10K0; Part Number (Vendor) (none) -> RMCF0201FT10K0TR-ND; SCH CHECK CHECKED -> SCH (N/A); Vendor (none) -> Digikey
- U401, U402: symbol _SCHLIB_Blender:BUF_SN74LVC1G17DBVR_SOT-23-5 -> _SCHLIB_Blender:IC_BUFFER_SN74LVC1G17DBVR_NON-INV_5.5V_0.032_SOT-23-5; Manufacturer (none) -> Texas Instruments; PCB CHECK (none) -> PCB (N/A); Package (none) -> SOT23-5; Part Number SN74LVC1G17DBVR -> (none); Part Number (Manufacturer) (none) -> SN74LVC1G17DBVR; Part Number (Vendor) (none) -> 296-11933-2-ND; SCH CHECK CHECKED -> SCH (N/A); Vendor (none) -> Digikey
Other:
- moved on the sheet: C401, C402, C403, C404, J401, J402, R401, R402, R403, R404, U401
