File: Hardware/Blender/v1_20230918/Design Folder/_HW_Blender/[05] - BUFFERED VGA INPUT.kicad_sch (KiCad schematic)
At the start: 21 parts, among them J501 DE-15_MALE_RA, U501 SN74LVC1G17DBVR, U502 SN74LVC1G17DBVR

Commit message: More update for hardware part
Parts:
- C501, C503: value 2u2F/6V3 -> 2u2F_6V3_X5R; symbol _SCHLIB_Blender:CAP_2u2F/6V3_C0201 -> _SCHLIB_Blender:CAP_2u2F_6V3_X5R_C0201; Manufacturer (none) -> KYOCERA AVX; PCB CHECk (none) -> PCB (N/A); Part Number CM03X5R225M06AH -> (none); Part Number (Manufacturer) (none) -> CM03X5R225M06AH; Part Number (Vendor) (none) -> 478-KGM03CR50J225MHTR-ND; SCH CHECK CHECKED -> SCH (N/A); Vendor (none) -> Digikey
- C502, C504: value 100nF/6V3 -> 100nF_6V3_X7R; symbol _SCHLIB_Blender:CAP_100nF/6V3_C0201 -> _SCHLIB_Blender:CAP_100nF_6V3_X7R_C0201; Manufacturer (none) -> YAGEO; PCB CHECk (none) -> PCB (N/A); Part Number CC0201KRX7R5BB104 -> (none); Part Number (Manufacturer) (none) -> CC0201KRX7R5BB104; Part Number (Vendor) (none) -> 13-CC0201KRX7R5BB104TR-ND; SCH CHECK CHECKED -> SCH (N/A); Vendor (none) -> Digikey
- D501, D502, D503, D504, D505: symbol _SCHLIB_Blender:TVS_GG040205100N2P_D0402 -> _SCHLIB_Blender:DIODE_TVS_GG040205100N2P_5V_5.5V_8A(8/20us)_D0402; IPP 8A (8/20us) -> (none); Manufacturer (none) -> KYOCERA AVX; PCB CHECk (none) -> PCB (N/A); Package (none) -> D0402; Part Number GG040205100N2P -> (none); Part Number (Manufacturer) (none) -> GG040205100N2P; Part Number (Vendor) (none) -> 478-10594-2-ND; SCH CHECK * -> SCH (N/A); VBR 5.5V (Vbr) -> (none); VC 12V (Vc) -> (none); Vendor (none) -> Digikey
- J501: value DE-15_MALE_RA -> DSUB_15POS_MALE_RA; symbol _SCHLIB_Blender:CONN_DE-15_MALE_RA -> _SCHLIB_Blender:CONN_DSUB_15POS_MALE_RA; Manufacturer (none) -> Amphenol ICC (Commercial Products); PCB CHECk (none) -> PCB (N/A); Package (none) -> THD-R/A; Part Number L717HDE15PD4CH4R -> (none); Part Number (Manufacturer) (none) -> L717HDE15PD4CH4R; Part Number (Vendor) (none) -> L717HDE15PD4CH4R-ND; SCH CHECK * -> SCH (N/A); Vendor (none) -> Digikey
- R501, R502, R503, R505, R508: value 75R_2W -> 75R_2W_1%; symbol _SCHLIB_Blender:RES_75R_2W_R1206 -> _SCHLIB_Blender:RES_75R_2W_1%_R1206; Manufacturer (none) -> TE Connectivity Passive Product; PCB CHECk (none) -> PCB (N/A); Part Number 3503G2B75RFTD -> (none); Part Number (Manufacturer) (none) -> 3503G2B75RFTD; Part Number (Vendor) (none) -> 1712-3503G2B75RFTDTR-ND; SCH CHECK * -> SCH (N/A); Vendor (none) -> Digikey
- R504, R507: value 10KR_1/20W -> 10KR_1/20W_1%; symbol _SCHLIB_Blender:RES_10KR_1/20W-R0201 -> _SCHLIB_Blender:RES_10KR_1/20W_1%_R0201; Manufacturer (none) -> Stackpole Electronics Inc; PCB CHECk (none) -> PCB (N/A); Part Number RMCF0201FT10K0 -> (none); Part Number (Manufacturer) (none) -> RMCF0201FT10K0; Part Number (Vendor) (none) -> RMCF0201FT10K0TR-ND; SCH CHECK CHECKED -> SCH (N/A); Vendor (none) -> Digikey
- R506, R509: value 49R9_1/20W -> 49R9_1/20W_1%; symbol _SCHLIB_Blender:RES_49R9_1/20W-R0201 -> _SCHLIB_Blender:RES_49R9_1/20W_1%_R0201; Manufacturer (none) -> Stackpole Electronics Inc; PCB CHECk (none) -> PCB (N/A); Part Number RMCF0201FT49R9 -> (none); Part Number (Manufacturer) (none) -> RMCF0201FT49R9; Part Number (Vendor) (none) -> RMCF0201FT49R9TR-ND; SCH CHECK CHECKED -> SCH (N/A); Vendor (none) -> Digikey
- U501, U502: symbol _SCHLIB_Blender:BUF_SN74LVC1G17DBVR_SOT-23-5 -> _SCHLIB_Blender:IC_BUFFER_SN74LVC1G17DBVR_NON-INV_5.5V_0.032_SOT-23-5; Manufacturer (none) -> Texas Instruments; PCB CHECK (none) -> PCB (N/A); Package (none) -> SOT23-5; Part Number SN74LVC1G17DBVR -> (none); Part Number (Manufacturer) (none) -> SN74LVC1G17DBVR; Part Number (Vendor) (none) -> 296-11933-2-ND; SCH CHECK CHECKED -> SCH (N/A); Vendor (none) -> Digikey
Other:
- moved on the sheet: C501, C502, C503, C504, D501, D502, D503, D504, D505, R504, R506, R507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
