File: Hardware/Blender/v1_20230918/Design Folder/_HW_Blender/[06] - ISOLATED WS28xx DRIVER.kicad_sch (KiCad schematic)
At the start: 41 parts, among them J601 MHDR_2POS_1.27MM_VERT, J602 RCPT_4POS_1.27MM, U601 SN74LVC1G17DBVR, U602 ISO7720FDR, U603 SN74LVC1G17DBVR, U604 DLPT05A-7, U605 DLPT05A-7

Commit message: Improving the file structure and documentation
Other:
- note removed: "UNCHECKED"
- moved on the sheet: C601, C602, C603, C604, C605, C606, C607, C608, C609, C610, C611, D601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

Commit message: More update for hardware part
Parts:
- C601, C602, C603, C604, C605, C606, C607, C608, C609, C611: value 2u2F/6V3 -> 2u2F_6V3_X5R; symbol _SCHLIB_Blender:CAP_2u2F/6V3_C0201 -> _SCHLIB_Blender:CAP_2u2F_6V3_X5R_C0201; Manufacturer (none) -> KYOCERA AVX; PCB CHECk (none) -> PCB (N/A); Part Number CM03X5R225M06AH -> (none); Part Number (Manufacturer) (none) -> CM03X5R225M06AH; Part Number (Vendor) (none) -> 478-KGM03CR50J225MHTR-ND; SCH CHECK CHECKED -> SCH (N/A); Vendor (none) -> Digikey
- C610: value 10uF/16V -> 10uF_16V_X5R; symbol _SCHLIB_Blender:CAP_10uF/16V-C0603 -> _SCHLIB_Blender:CAP_10uF_16V_X5R_C0603; Manufacturer (none) -> Murata Electronics; PCB CHECk (none) -> PCB (N/A); Part Number GRT188R61C106KE13J -> (none); Part Number (Manufacturer) (none) -> GRT188R61C106KE13J; Part Number (Vendor) (none) -> 490-GRT188R61C106KE13JTR-ND; SCH CHECK CHECKED -> SCH (N/A); Vendor (none) -> Digikey
- D601, D602, D603, D604, D605, D606, D607: symbol _SCHLIB_Blender:LED_WS2812B_5050 -> _SCHLIB_Blender:IC_LED_WS2812B_RGB_5V_0.06A_PLCC4-5050; Manufacturer (none) -> SparkFun Electronics; PCB CHECk (none) -> PCB (N/A); Package (none) -> PLCC4-5050; Part Number COM-16347 -> (none); Part Number (Manufacturer) (none) -> COM-16347; Part Number (Vendor) (none) -> 1568-COM-16347TR-ND; SCH CHECK * -> SCH (N/A); Vendor (none) -> Digikey
- J601: value MHDR_2POS_1.27MM_VERT -> MHDR_2X1_VERT_1.27MM; symbol _SCHLIB_Blender:CONN_MHDR_2POS_1.27MM_VERT -> _SCHLIB_Blender:CONN_HEADER_2POS_1ROW_MALE_VERT_1.27MM; Manufacturer (none) -> Sullins Connector Solutions; PCB CHECk (none) -> PCB (N/A); Package (none) -> THD-RA-2.54MM; Part Number GRPB021VWVN-RC -> (none); Part Number (Manufacturer) (none) -> GRPB021VWVN-RC; Part Number (Vendor) (none) -> S9014E-02-ND; SCH CHECK CHECKED -> SCH (N/A); Vendor (none) -> Digikey
- J602: value RCPT_4POS_1.27MM -> RECEPT_4X1_VERT_1.27MM; symbol _SCHLIB_Blender:CONN_RCPT_4POS_1.27MM_VERT -> _SCHLIB_Blender:CONN_RECEPT_4POS_1ROW_VERT_1.27MM; Manufacturer (none) -> GCT; PCB CHECk (none) -> PCB (N/A); Package (none) -> THD-VERT-2.54MM; Part Number BD080-04-A-0230-L-D -> (none); Part Number (Manufacturer) (none) -> BD080-04-A-0230-L-D; Part Number (Vendor) (none) -> 2073-BD080-04-A-0230-L-D-ND; SCH CHECK CHECKED -> SCH (N/A); Vendor (none) -> Digikey
- LED601: value GREEN -> GREEN_2V8; symbol _SCHLIB_Blender:LED_GREEN_0402 -> _SCHLIB_Blender:DIODE_LED_GREEN_2.8V_0.02A_529nm_0402; Manufacturer (none) -> Harvatek Corporation; PCB CHECk (none) -> PCB (N/A); Part Number B2841NG--05D000514U1930 -> (none); Part Number (Manufacturer) (none) -> B2841NG--05D000514U1930; Part Number (Vendor) (none) -> 3147-B2841NG--05D000514U1930TR-ND; SCH CHECK CHECKED -> SCH (N/A); VOLTAGE RATED 2V8 -> (none); Vendor (none) -> Digikey
- R601, R602, R603, R605, R606, R607, R608, R610, R613, R614: value 100R_1/20W -> 100R_1/20W_1%; symbol _SCHLIB_Blender:RES_100R_1/20W-R0201 -> _SCHLIB_Blender:RES_100R_1/20W_1%_R0201; Manufacturer (none) -> Stackpole Electronics Inc; PCB CHECk (none) -> PCB (N/A); Part Number RMCF0201FT100R -> (none); Part Number (Manufacturer) (none) -> RMCF0201FT100R; Part Number (Vendor) (none) -> RMCF0201FT100RTR-ND; SCH CHECK CHECKED -> SCH (N/A); Vendor (none) -> Digikey
- R604: value 10KR_1/20W -> 10KR_1/20W_1%; symbol _SCHLIB_Blender:RES_10KR_1/20W-R0201 -> _SCHLIB_Blender:RES_10KR_1/20W_1%_R0201; Manufacturer (none) -> Stackpole Electronics Inc; PCB CHECk (none) -> PCB (N/A); Part Number RMCF0201FT10K0 -> (none); Part Number (Manufacturer) (none) -> RMCF0201FT10K0; Part Number (Vendor) (none) -> RMCF0201FT10K0TR-ND; SCH CHECK CHECKED -> SCH (N/A); Vendor (none) -> Digikey
- R609: value 100R_1/8W -> 100R_1/8W_5%; symbol _SCHLIB_Blender:RES_100R_1/8W_R0805 -> _SCHLIB_Blender:RES_100R_1/8W_5%_R0805; Manufacturer (none) -> TE Connectivity Passive Product; PCB CHECk (none) -> PCB (N/A); Part Number CRGCQ0805J100R -> (none); Part Number (Manufacturer) (none) -> CRGCQ0805J100R; Part Number (Vendor) (none) -> A130128TR-ND; SCH CHECK * -> SCH (N/A); Vendor (none) -> Digikey
- R611, R612: value 1KR_1/8W -> 1KR_1/8W_5%; symbol _SCHLIB_Blender:RES_1KR_1/8W_R0805 -> _SCHLIB_Blender:RES_1KR_1/8W_5%_R0805; Manufacturer (none) -> TE Connectivity Passive Product; PCB CHECk (none) -> PCB (N/A); Part Number CRGCQ0805J1K0 -> (none); Part Number (Manufacturer) (none) -> CRGCQ0805J1K0; Part Number (Vendor) (none) -> A130134TR-ND; SCH CHECK * -> SCH (N/A); Vendor (none) -> Digikey
- R615: value 470R_1/16W -> 470R_1/16W_5%; symbol _SCHLIB_Blender:RES_470R_1/16W_R0402 -> _SCHLIB_Blender:RES_470R_1/16W_5%_R0402; Manufacturer (none) -> TE Connectivity Passive Product; PCB CHECk (none) -> PCB (N/A); Part Number CRGCQ0402J470R -> (none); Part Number (Manufacturer) (none) -> CRGCQ0402J470R; Part Number (Vendor) (none) -> A130046TR-ND; SCH CHECK * -> SCH (N/A); Vendor (none) -> Digikey
- U601, U603: symbol _SCHLIB_Blender:BUF_SN74LVC1G17DBVR_SOT-23-5 -> _SCHLIB_Blender:IC_BUFFER_SN74LVC1G17DBVR_NON-INV_5.5V_0.032_SOT-23-5; Manufacturer (none) -> Texas Instruments; PCB CHECK (none) -> PCB (N/A); Package (none) -> SOT23-5; Part Number SN74LVC1G17DBVR -> (none); Part Number (Manufacturer) (none) -> SN74LVC1G17DBVR; Part Number (Vendor) (none) -> 296-11933-2-ND; SCH CHECK CHECKED -> SCH (N/A); Vendor (none) -> Digikey
- U602: symbol _SCHLIB_Blender:IC_ISO7720FDR -> _SCHLIB_Blender:IC_ISOLATOR_ISO7720FDR_3000Vrms_100Mbps_8-SOIC (0.154{dblquote}, 3.90mm Width); Manufacturer (none) -> Texas Instruments; PCB CHECk (none) -> PCB (N/A); Package (none) -> 8-SOIC (0.154", 3.90mm Width); Part Number ISO7720FDR -> (none); Part Number (Manufacturer) (none) -> ISO7720FDR; Part Number (Vendor) (none) -> 296-51198-2-ND; SCH CHECK CHECKED -> SCH (N/A); Vendor (none) -> Digikey
- U604, U605: symbol _SCHLIB_Blender:TVS_DLPT05A-7_SOT_23 -> _SCHLIB_Blender:DIODE_TVS_DLPT05A-7_5V_6V_17A(8/20us)_SOT_23-3; C@F 1.9pF@1MHz -> (none); Ipp 17A (Ipp 8/20uS) -> (none); Manufacturer (none) -> Diodes Incorporated; PCB CHECk (none) -> PCB (N/A); Package (none) -> SOT-23-3; Part Number DLPT05A-7 -> (none); Part Number (Manufacturer) (none) -> DLPT05A-7; Part Number (Vendor) (none) -> 31-DLPT05A-7TR-ND; SCH CHECK CHECKED -> SCH (N/A); Vbr 6 (Vbr) -> (none); Vc 9.8 (Vc) -> (none); Vendor (none) -> Digikey
Other:
- moved on the sheet: C601, C602, C603, C604, C605, C606, C607, C608, C609, C610, C611, D601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
