File: Hardware/Blender/v1_20230918/Design Folder/_HW_Blender/[07] - ISOLATED DMX.kicad_sch (KiCad schematic)
At the start: 22 parts, among them J701 RCPT_3POS_1.27MM, U701 1S4E_0505S1.5U, U702 SN74LVC1G17DBVR, U703 CDSOT23-SM712, U704 MAX22028AWA+, U705 SN74LVC1G17DBVR

Commit message: Improving the file structure and documentation
Other:
- note removed: "UNCHECKED"
- moved on the sheet: C701, C702, C703, C704, C705, C706, F701, F702, F703, J701, LED701, R701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

Commit message: More update for hardware part
Parts:
- C701, C702, C703, C704, C705, C706: value 10uF/16V -> 10uF_16V_X5R; symbol _SCHLIB_Blender:CAP_10uF/16V-C0603 -> _SCHLIB_Blender:CAP_10uF_16V_X5R_C0603; Manufacturer (none) -> Murata Electronics; PCB CHECk (none) -> PCB (N/A); Part Number GRT188R61C106KE13J -> (none); Part Number (Manufacturer) (none) -> GRT188R61C106KE13J; Part Number (Vendor) (none) -> 490-GRT188R61C106KE13JTR-ND; SCH CHECK CHECKED -> SCH (N/A); Vendor (none) -> Digikey
- F701, F702, F703: value 0805L010/24YR -> 0.1A_24V_1.5R; symbol _SCHLIB_Blender:PTC_0805L010/24YR_F0805 -> _SCHLIB_Blender:FUSE_PTC_0805L010/24YR_0.1A_0.3A_24V_F0805; Ihold 100 mA -> (none); Manufacturer (none) -> Littelfuse Inc.; PCB CHECk (none) -> PCB (N/A); Part Number 0805L010/24YR -> (none); Part Number (Manufacturer) (none) -> 0805L010/24YR; Part Number (Vendor) (none) -> F11311TR-ND; SCH CHECK CHECKED -> SCH (N/A); Vendor (none) -> Digikey; Voltage Rated 24 V -> (none)
- J701: value RCPT_3POS_1.27MM -> RECEPT_3X1_VERT_1.27MM; symbol _SCHLIB_Blender:CONN_RCPT_3POS_1.27MM_VERT -> _SCHLIB_Blender:CONN_RECEPT_3POS_1ROW_VERT_1.27MM; Manufacturer (none) -> GCT; PCB CHECk (none) -> PCB (N/A); Package (none) -> THD-VERT-2.54MM; Part Number BD080-03-A-0230-L-G -> (none); Part Number (Manufacturer) (none) -> BD080-03-A-0230-L-G; Part Number (Vendor) (none) -> 2073-BD080-03-A-0230-L-G-ND; SCH CHECK CHECKED -> SCH (N/A); Vendor (none) -> Digikey
- LED701: value GREEN -> GREEN_2V8; symbol _SCHLIB_Blender:LED_GREEN_0402 -> _SCHLIB_Blender:DIODE_LED_GREEN_2.8V_0.02A_529nm_0402; Manufacturer (none) -> Harvatek Corporation; PCB CHECk (none) -> PCB (N/A); Part Number B2841NG--05D000514U1930 -> (none); Part Number (Manufacturer) (none) -> B2841NG--05D000514U1930; Part Number (Vendor) (none) -> 3147-B2841NG--05D000514U1930TR-ND; SCH CHECK CHECKED -> SCH (N/A); VOLTAGE RATED 2V8 -> (none); Vendor (none) -> Digikey
- R701: value 470R_1/16W -> 470R_1/16W_5%; symbol _SCHLIB_Blender:RES_470R_1/16W_R0402 -> _SCHLIB_Blender:RES_470R_1/16W_5%_R0402; Manufacturer (none) -> TE Connectivity Passive Product; PCB CHECk (none) -> PCB (N/A); Part Number CRGCQ0402J470R -> (none); Part Number (Manufacturer) (none) -> CRGCQ0402J470R; Part Number (Vendor) (none) -> A130046TR-ND; SCH CHECK * -> SCH (N/A); Vendor (none) -> Digikey
- R702: value 10KR_1/20W -> 10KR_1/20W_1%; symbol _SCHLIB_Blender:RES_10KR_1/20W-R0201 -> _SCHLIB_Blender:RES_10KR_1/20W_1%_R0201; Manufacturer (none) -> Stackpole Electronics Inc; PCB CHECk (none) -> PCB (N/A); Part Number RMCF0201FT10K0 -> (none); Part Number (Manufacturer) (none) -> RMCF0201FT10K0; Part Number (Vendor) (none) -> RMCF0201FT10K0TR-ND; SCH CHECK CHECKED -> SCH (N/A); Vendor (none) -> Digikey
- R703, R706: value 680R_1/8W -> 680R_1/8W_5%; symbol _SCHLIB_Blender:RES_680R_1/8W_R0805 -> _SCHLIB_Blender:RES_680R_1/8W_5%_R0805; Manufacturer (none) -> Stackpole Electronics Inc; PCB CHECk (none) -> PCB (N/A); Part Number RMCF0805JT680R -> (none); Part Number (Manufacturer) (none) -> RMCF0805JT680R; Part Number (Vendor) (none) -> RMCF0805JT680RTR-ND; SCH CHECK CHECKED -> SCH (N/A); Vendor (none) -> Digikey
- R704, R705: value 100R_1/20W -> 100R_1/20W_1%; symbol _SCHLIB_Blender:RES_100R_1/20W-R0201 -> _SCHLIB_Blender:RES_100R_1/20W_1%_R0201; Manufacturer (none) -> Stackpole Electronics Inc; PCB CHECk (none) -> PCB (N/A); Part Number RMCF0201FT100R -> (none); Part Number (Manufacturer) (none) -> RMCF0201FT100R; Part Number (Vendor) (none) -> RMCF0201FT100RTR-ND; SCH CHECK CHECKED -> SCH (N/A); Vendor (none) -> Digikey
- U701: symbol _SCHLIB_Blender:DCDC_1S4E_0505S1.5U -> _SCHLIB_Blender:IC_PMIC_1S4E_0505S1.5U_ISO-DCDC_5IN_5OUT_0.2A_4SIP; Manufacturer (none) -> GAPTEC Electronic; PCB CHECk (none) -> PCB (N/A); Package (none) -> 4-SIP Module; Part Number 1S4E_0505S1.5U -> (none); Part Number (Manufacturer) (none) -> 1S4E_0505S1.5U; Part Number (Vendor) (none) -> 3182-1S4E_0505S1.5U-ND; SCH CHECK * -> SCH (N/A); Vendor (none) -> Digikey
- U702, U705: symbol _SCHLIB_Blender:BUF_SN74LVC1G17DBVR_SOT-23-5 -> _SCHLIB_Blender:IC_BUFFER_SN74LVC1G17DBVR_NON-INV_5.5V_0.032_SOT-23-5; Manufacturer (none) -> Texas Instruments; PCB CHECK (none) -> PCB (N/A); Package (none) -> SOT23-5; Part Number SN74LVC1G17DBVR -> (none); Part Number (Manufacturer) (none) -> SN74LVC1G17DBVR; Part Number (Vendor) (none) -> 296-11933-2-ND; SCH CHECK CHECKED -> SCH (N/A); Vendor (none) -> Digikey
- U703: symbol _SCHLIB_Blender:TVS_CDSOT23-SM712 -> _SCHLIB_Blender:DIODE_TVS_CDSOT23-SM712_12V_13.3V_17A(8/20us)_SOT-23-3; Manufacturer (none) -> Bourns Inc.; PCB CHECk (none) -> PCB (N/A); Package (none) -> SOT-23-3; Part Number CDSOT23-SM712 -> (none); Part Number (Manufacturer) (none) -> CDSOT23-SM712; Part Number (Vendor) (none) -> CDSOT23-SM712TR-ND; SCH CHECK * -> SCH (N/A); Vendor (none) -> Digikey
- U704: symbol _SCHLIB_Blender:IC_MAX22028AWA+ -> _SCHLIB_Blender:IC_ISOLATOR_MAX22028AWA+_RS485_8-SOIC (0.209{dblquote}, 5.30mm Width); Manufacturer (none) -> Analog Devices Inc./Maxim Integrated; PCB CHECk (none) -> PCB (N/A); Package (none) -> 8-SOIC (0.209", 5.30mm Width); Part Number MAX22028FAWA+ -> (none); Part Number (Manufacturer) (none) -> MAX22028FAWA+; Part Number (Vendor) (none) -> 175-MAX22028AWA+-ND; SCH CHECK CHECKED -> SCH (N/A); Vendor (none) -> Digikey
Other:
- moved on the sheet: C703, C704, C705, C706, F701, F702, F703, J701, LED701, R701, R702, R703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
