File: Hardware/Blender/v1_20230918/Design Folder/_HW_Blender/[08] - SPEAKER DRIVER.kicad_sch (KiCad schematic)
At the start: 27 parts, among them J801 MHDR_2POS_1.27MM_VERT, J802 MHDR_2POS_1.27MM_VERT, U801 PAM8003DR, U802 PCM1754DBQR

Commit message: Improving the file structure and documentation
Other:
- note removed: "UNCHECKED"
- moved on the sheet: C801, C802, C803, C804, C805, C806, C807, C808, J801, J802, R801, R802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

Commit message: More update for hardware part
Parts:
- C801, C802, C803, C804: value 10uF/16V -> 10uF_16V_X5R; symbol _SCHLIB_Blender:CAP_10uF/16V-C0603 -> _SCHLIB_Blender:CAP_10uF_16V_X5R_C0603; Manufacturer (none) -> Murata Electronics; PCB CHECk (none) -> PCB (N/A); Part Number GRT188R61C106KE13J -> (none); Part Number (Manufacturer) (none) -> GRT188R61C106KE13J; Part Number (Vendor) (none) -> 490-GRT188R61C106KE13JTR-ND; SCH CHECK CHECKED -> SCH (N/A); Vendor (none) -> Digikey
- C805, C806, C808: value 2u2F/6V3 -> 2u2F_6V3_X5R; symbol _SCHLIB_Blender:CAP_2u2F/6V3_C0201 -> _SCHLIB_Blender:CAP_2u2F_6V3_X5R_C0201; Manufacturer (none) -> KYOCERA AVX; PCB CHECk (none) -> PCB (N/A); Part Number CM03X5R225M06AH -> (none); Part Number (Manufacturer) (none) -> CM03X5R225M06AH; Part Number (Vendor) (none) -> 478-KGM03CR50J225MHTR-ND; SCH CHECK CHECKED -> SCH (N/A); Vendor (none) -> Digikey
- C807: value 1uF/6V3 -> 1uF_6V3_X5R; symbol _SCHLIB_Blender:CAP_1uF/6V3_C0201 -> _SCHLIB_Blender:CAP_1uF_6V3_X5R_C0201; Manufacturer (none) -> Samsung Electro-Mechanics; PCB CHECk (none) -> PCB (N/A); Part Number CL03A105MQ3CSNH -> (none); Part Number (Manufacturer) (none) -> CL03A105MQ3CSNH; Part Number (Vendor) (none) -> 1276-6441-2-ND; SCH CHECK CHECKED -> SCH (N/A); Vendor (none) -> Digikey
- J801, J802: value MHDR_2POS_1.27MM_VERT -> MHDR_2X1_VERT_1.27MM; symbol _SCHLIB_Blender:CONN_MHDR_2POS_1.27MM_VERT -> _SCHLIB_Blender:CONN_HEADER_2POS_1ROW_MALE_VERT_1.27MM; Manufacturer (none) -> Sullins Connector Solutions; PCB CHECk (none) -> PCB (N/A); Package (none) -> THD-RA-2.54MM; Part Number GRPB021VWVN-RC -> (none); Part Number (Manufacturer) (none) -> GRPB021VWVN-RC; Part Number (Vendor) (none) -> S9014E-02-ND; SCH CHECK CHECKED -> SCH (N/A); Vendor (none) -> Digikey
- R801: value 10KR_1/20W -> 10KR_1/20W_1%; symbol _SCHLIB_Blender:RES_10KR_1/20W-R0201 -> _SCHLIB_Blender:RES_10KR_1/20W_1%_R0201; Manufacturer (none) -> Stackpole Electronics Inc; PCB CHECk (none) -> PCB (N/A); Part Number RMCF0201FT10K0 -> (none); Part Number (Manufacturer) (none) -> RMCF0201FT10K0; Part Number (Vendor) (none) -> RMCF0201FT10K0TR-ND; SCH CHECK CHECKED -> SCH (N/A); Vendor (none) -> Digikey
- R802: value 100R_1/10W -> 100R_1/10W_1%; symbol _SCHLIB_Blender:RES_100R_1/10W_R0402 -> _SCHLIB_Blender:RES_100R_1/10W_1%_R0402; Manufacturer (none) -> Panasonic Electronic Components; PCB CHECk (none) -> PCB (N/A); Part Number ERJ-2RKF1000X -> (none); Part Number (Manufacturer) (none) -> ERJ-2RKF1000X; Part Number (Vendor) (none) -> P100LTR-ND; SCH CHECK * -> SCH (N/A); Vendor (none) -> Digikey
- R803, R804, R805, R806, R807, R808, R809, R810, R811: value 100R_1/20W -> 100R_1/20W_1%; symbol _SCHLIB_Blender:RES_100R_1/20W-R0201 -> _SCHLIB_Blender:RES_100R_1/20W_1%_R0201; Manufacturer (none) -> Stackpole Electronics Inc; PCB CHECk (none) -> PCB (N/A); Part Number RMCF0201FT100R -> (none); Part Number (Manufacturer) (none) -> RMCF0201FT100R; Part Number (Vendor) (none) -> RMCF0201FT100RTR-ND; SCH CHECK CHECKED -> SCH (N/A); Vendor (none) -> Digikey
- R812, R813, R814, R815: value 4K7R_1/20W -> 47KR_1/20W_1%; symbol _SCHLIB_Blender:RES_4K7R_1/20W-R0201 -> _SCHLIB_Blender:RES_47KR_1/20W_1%_R0201; Link https://www.digikey.ca/en/products/detail/stackpole-electro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 -> https://www.digikey.ca/en/products/detail/yageo/AC0201FR-07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; Manufacturer (none) -> YAGEO; PCB CHECk (none) -> PCB (N/A); Part Number RMCF0201FT4K70 -> (none); Part Number (Manufacturer) (none) -> AC0201FR-0747KL; Part Number (Vendor) (none) -> YAG3425TR-ND; SCH CHECK CHECKED -> SCH (N/A); Vendor (none) -> Digikey
- U801: symbol _SCHLIB_Blender:AMP_PAM8003DR -> _SCHLIB_Blender:IC_AMP_PAM8003DR_STEREO_CLASS D_16-SOIC (0.154{dblquote}, 3.90mm Width); Manufacturer (none) -> Diodes Incorporated; PCB CHECK (none) -> PCB (N/A); Package (none) -> 16-SOIC (0.154", 3.90mm Width); Part Number (Vendor) (none) -> PAM8003DRDITR-ND; SCH CHECK * -> SCH (N/A); Vendor (none) -> Digikey
- U802: symbol _SCHLIB_Blender:IC_PCM1754DBQR -> _SCHLIB_Blender:IC_DAC_PCM1754DBQR_24b_I2S_16SSOP; Manufacturer (none) -> Texas Instruments; PCB CHECk (none) -> PCB (N/A); Package (none) -> 16-SSOP (0.154", 3.90mm Width); Part Number PCM1754DBQR -> (none); Part Number (Manufacturer) (none) -> PCM1754DBQR; Part Number (Vendor) (none) -> 296-26302-2-ND; SCH CHECK * -> SCH (N/A); Vendor (none) -> Digikey
Connections:
- net PAM8003_VOLUME: now also R802.2, U801.12 (VOLUME)
- net PCM_SCK: now reaches R811.2, R812.1, U802.16 (SCK)
- net PAM8003_INL: now reaches R805.2, U801.7 (INL)
- net PCM_MUTE: now reaches R803.2, U802.14 (MUTE)
- net PCM_DATA: now reaches R809.2, R814.1, U802.2 (DATA)
- net PCM_DEMP: now reaches R806.2, U802.13 (DEMP)
- net PCM_BCK: now reaches R810.2, R813.1, U802.1 (BCK)
- net PCM_FMT: now reaches R804.2, U802.15 (FMT)
- net PCM_LRCK: now reaches R808.2, R815.1, U802.3 (LRCK)
- net PCM_L_OUT: now reaches C801.1, U802.7 (V_L_OUT)
- net PCM_R_OUT: now reaches C802.1, U802.8 (V_R_OUT)
- net PAM8003_INR: now reaches R807.2, U801.10 (INR)
- net SPKL+ renamed PAM8003_SPKL+
- net SPKL- renamed PAM8003_SPKL-
- net SPKR+ renamed PAM8003_SPKR+
- net SPKR- renamed PAM8003_SPKR-
Other:
- moved on the sheet: C801, C802, C803, C804, C805, C806, C807, C808, J801, J802, R801, R802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
