File: Hardware/Blender/v1_20230918/Design Folder/_HW_Blender/[10] - Power Supply.kicad_sch (KiCad schematic)
At the start: 36 parts, among them J1001 MHDR_2POS_1.27MM_VERT, J1002 MICRO B USB_RA, Q1001 SI4455DY-T1-GE3, Q1002 RN1130MFV,L3F, U1001 TPS613222ADBVR, U1002 TLV74033PDBVR, U1003 MCP73811T-420I/OT, U1004 TLV74033PDBVR

Commit message: Improving the file structure and documentation
Other:
- note added: "DESIGN NOTE:"
- note added: "The high switching frequency of TPS61322xx demands a high-speed rectifying switch for optimum efficiency. Ensure that the average and peak current rating of the diode exceeds the average output current and peak inductor current. In addition, the reverse breakdown voltage of the diode must exceed the maximum output voltage of the converter. A snubber circuit consisting of a resistor R1 and a capac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"
- note removed: "DESIGN NOTE: The high switching frequency of TPS61322xx demands a high-speed rectifying switch for optimum efficiency. Ensure that the average and peak current rating of the diode exceeds the average output current and peak inductor current. In addition, the reverse breakdown voltage of the diode must exceed the maximum output voltage of the converter. A snubber circuit consisting of a resistor R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"
- note removed: "UNCHECKED"
- moved on the sheet: C1001, C1002, C1003, C1004, C1005, C1006, C1007, C1008, C1009, C1010, D1001, D1002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

Commit message: More update for hardware part
Parts:
- C1001: value 680pF_50V -> 680pF_50V_X7R; symbol _SCHLIB_Blender:CAP_680pF_50V_C0402 -> _SCHLIB_Blender:CAP_680pF_50V_X7R_C0402; Manufacturer (none) -> Walsin Technology Corporation; PCB CHECk (none) -> PCB (N/A); Part Number 0402B681K500CT -> (none); Part Number (Manufacturer) (none) -> 0402B681K500CT; Part Number (Vendor) (none) -> 1292-1223-2-ND; SCH CHECK * -> SCH (N/A); Vendor (none) -> Digikey
- C1002, C1003, C1004, C1007, C1008, C1009, C1010: value 10uF/16V -> 10uF_16V_X5R; symbol _SCHLIB_Blender:CAP_10uF/16V-C0603 -> _SCHLIB_Blender:CAP_10uF_16V_X5R_C0603; Manufacturer (none) -> Murata Electronics; PCB CHECk (none) -> PCB (N/A); Part Number GRT188R61C106KE13J -> (none); Part Number (Manufacturer) (none) -> GRT188R61C106KE13J; Part Number (Vendor) (none) -> 490-GRT188R61C106KE13JTR-ND; SCH CHECK CHECKED -> SCH (N/A); Vendor (none) -> Digikey
- C1005, C1006: value 1uF/6V3 -> 1uF_6V3_X5R; symbol _SCHLIB_Blender:CAP_1uF/6V3_C0201 -> _SCHLIB_Blender:CAP_1uF_6V3_X5R_C0201; Manufacturer (none) -> Samsung Electro-Mechanics; PCB CHECk (none) -> PCB (N/A); Part Number CL03A105MQ3CSNH -> (none); Part Number (Manufacturer) (none) -> CL03A105MQ3CSNH; Part Number (Vendor) (none) -> 1276-6441-2-ND; SCH CHECK CHECKED -> SCH (N/A); Vendor (none) -> Digikey
- D1001: symbol _SCHLIB_Blender:SCHOTTKY_SK510A-LTP_SMA -> _SCHLIB_Blender:DIODE_SCHOTTKY_SK510A-LTP_5A_100V_SMA; C 200pF @ 4V/1MHz -> (none); Io 5A -> (none); Manufacturer (none) -> Micro Commercial Co; PCB CHECk (none) -> PCB (N/A); Part Number SK510A-LTP -> (none); Part Number (Manufacturer) (none) -> SK510A-LTP; Part Number (Vendor) (none) -> SK510A-LTPMSTR-ND; SCH CHECK * -> SCH (N/A); Vendor (none) -> Digikey; Vr 100V -> (none)
- D1002, D1003: symbol _SCHLIB_Blender:TVS_GG040205100N2P_D0402 -> _SCHLIB_Blender:DIODE_TVS_GG040205100N2P_5V_5.5V_8A(8/20us)_D0402; IPP 8A (8/20us) -> (none); Manufacturer (none) -> KYOCERA AVX; PCB CHECk (none) -> PCB (N/A); Package (none) -> D0402; Part Number GG040205100N2P -> (none); Part Number (Manufacturer) (none) -> GG040205100N2P; Part Number (Vendor) (none) -> 478-10594-2-ND; SCH CHECK * -> SCH (N/A); VBR 5.5V (Vbr) -> (none); VC 12V (Vc) -> (none); Vendor (none) -> Digikey
- F1001: value 0ZCK0100FF2E -> 1A_6V_0.06R; symbol _SCHLIB_Blender:PTC_0ZCK0100FF2E_F0805 -> _SCHLIB_Blender:FUSE_PTC_0ZCK0100FF2E_1A_1.95A_6V_F0805; Ih 1A -> (none); Manufacturer (none) -> Bel Fuse Inc.; PCB CHECk (none) -> PCB (N/A); Part Number 0ZCK0100FF2E -> (none); Part Number (Manufacturer) (none) -> 0ZCK0100FF2E; Part Number (Vendor) (none) -> 507-1815-2-ND; SCH CHECK CHECKED -> SCH (N/A); Vendor (none) -> Digikey; Vmax 6V -> (none)
- J1001: value MHDR_2POS_1.27MM_VERT -> MHDR_2X1_VERT_1.27MM; symbol _SCHLIB_Blender:CONN_MHDR_2POS_1.27MM_VERT -> _SCHLIB_Blender:CONN_HEADER_2POS_1ROW_MALE_VERT_1.27MM; Manufacturer (none) -> Sullins Connector Solutions; PCB CHECk (none) -> PCB (N/A); Package (none) -> THD-RA-2.54MM; Part Number GRPB021VWVN-RC -> (none); Part Number (Manufacturer) (none) -> GRPB021VWVN-RC; Part Number (Vendor) (none) -> S9014E-02-ND; SCH CHECK CHECKED -> SCH (N/A); Vendor (none) -> Digikey
- J1002: Manufacturer (none) -> Amphenol ICC (FCI); PCB CHECk (none) -> PCB (N/A); Package (none) -> SMD-RA; Part Number 10118194-0001LF -> (none); Part Number (Manufacturer) (none) -> 10118194-0001LF; Part Number (Vendor) (none) -> 609-4618-2-ND; SCH CHECK CHECKED -> SCH (N/A); Vendor (none) -> Digikey
- L1001: value 2u2H_2A -> 2u2H_2A_0.14R; symbol _SCHLIB_Blender:IND_2u2H_2A -> _SCHLIB_Blender:IND_2u2H__2A_0.14R_60MHz_L0806; DCR 140 mOhm -> (none); Manufacturer (none) -> INPAQ Technology Co., Ltd; PCB CHECk (none) -> PCB (N/A); Part Number WIP201610S-2R2MLDG -> (none); Part Number (Manufacturer) (none) -> WIP201610S-2R2MLDG; Part Number (Vendor) (none) -> 3526-WIP201610S-2R2MLDGCT-ND; SCH CHECK * -> SCH (N/A); Vendor (none) -> Digikey
- LED1001: value GREEN -> GREEN_2V8; symbol _SCHLIB_Blender:LED_GREEN_0402 -> _SCHLIB_Blender:DIODE_LED_GREEN_2.8V_0.02A_529nm_0402; Manufacturer (none) -> Harvatek Corporation; PCB CHECk (none) -> PCB (N/A); Part Number B2841NG--05D000514U1930 -> (none); Part Number (Manufacturer) (none) -> B2841NG--05D000514U1930; Part Number (Vendor) (none) -> 3147-B2841NG--05D000514U1930TR-ND; SCH CHECK CHECKED -> SCH (N/A); VOLTAGE RATED 2V8 -> (none); Vendor (none) -> Digikey
- LED1002, LED1003: value AMBER -> AMBER_2V; symbol _SCHLIB_Blender:LED_AMBER_0402 -> _SCHLIB_Blender:DIODE_LED_AMBER_2V_0.02A_592nm_0402; Manufacturer (none) -> Harvatek Corporation; PCB CHECk (none) -> PCB (N/A); Part Number B2841UY--20D000414U1930 -> (none); Part Number (Manufacturer) (none) -> B2841UY--20D000414U1930; Part Number (Vendor) (none) -> 3147-B2841UY--20D000414U1930TR-ND; SCH CHECK CHECKED -> SCH (N/A); VOLTAGE RATED 2V -> (none); Vendor (none) -> Digikey
- Q1001: symbol _SCHLIB_ToslinkToDMX:Q_SI4455DY-T1-GE3 -> _SCHLIB_Blender:Q_MOSFET_SI4455DY-T1-GE3_P-CH_150V_2A_5.9W_8-SOIC (0.154{dblquote}, 3.90mm Width); Manufacturer (none) -> Vishay Siliconix; PCB CHECk (none) -> PCB (N/A); Package (none) -> 8-SOIC (0.154", 3.90mm Width); Part Number SI4455DY-T1-GE3 -> (none); Part Number (Manufacturer) (none) -> SI4455DY-T1-GE3; Part Number (Vendor) (none) -> SI4455DY-T1-GE3TR-ND; SCH CHECK * -> SCH (N/A); Vendor (none) -> Digikey
- Q1002: symbol _SCHLIB_ToslinkToDMX:Q_RN1130MFV,L3F -> _SCHLIB_Blender:Q_BJT_RN1130MFV,L3F_PREBIASED_50V_0.1A_0.15W_SOT-723; Manufacturer (none) -> Toshiba Semiconductor and Storage; PCB CHECk (none) -> PCB (N/A); Part Number RN1130MFV,L3F -> (none); Part Number (Manufacturer) (none) -> RN1130MFV,L3F; Part Number (Vendor) (none) -> RN1130MFVL3FTR-ND; SCH CHECK * -> SCH (N/A); Vendor (none) -> Digikey
- R1001: value 4R7_1/4W -> 4R7_1/4W_1%; symbol _SCHLIB_Blender:RES_4R7_1/4W_R0805 -> _SCHLIB_Blender:RES_4R7_1/4W_1%_R0805; Manufacturer (none) -> KOA Speer Electronics, Inc.; PCB CHECk (none) -> PCB (N/A); Part Number RK73H2ATTD4R70F -> (none); Part Number (Manufacturer) (none) -> RK73H2ATTD4R70F; Part Number (Vendor) (none) -> 2019-RK73H2ATTD4R70FTR-ND; SCH CHECK * -> SCH (N/A); Vendor (none) -> Digikey
- R1002: value 4K7R_1/20W -> 47KR_1/20W_1%; symbol _SCHLIB_Blender:RES_4K7R_1/20W-R0201 -> _SCHLIB_Blender:RES_47KR_1/20W_1%_R0201; Link https://www.digikey.ca/en/products/detail/stackpole-electro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 -> https://www.digikey.ca/en/products/detail/yageo/AC0201FR-07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; Manufacturer (none) -> YAGEO; PCB CHECk (none) -> PCB (N/A); Part Number RMCF0201FT4K70 -> (none); Part Number (Manufacturer) (none) -> AC0201FR-0747KL; Part Number (Vendor) (none) -> YAG3425TR-ND; SCH CHECK CHECKED -> SCH (N/A); Vendor (none) -> Digikey
- R1003, R1005, R1008: value 470R_1/16W -> 470R_1/16W_5%; symbol _SCHLIB_Blender:RES_470R_1/16W_R0402 -> _SCHLIB_Blender:RES_470R_1/16W_5%_R0402; Manufacturer (none) -> TE Connectivity Passive Product; PCB CHECk (none) -> PCB (N/A); Part Number CRGCQ0402J470R -> (none); Part Number (Manufacturer) (none) -> CRGCQ0402J470R; Part Number (Vendor) (none) -> A130046TR-ND; SCH CHECK * -> SCH (N/A); Vendor (none) -> Digikey
- R1004, R1007: value 10KR_1/20W -> 10KR_1/20W_1%; symbol _SCHLIB_Blender:RES_10KR_1/20W-R0201 -> _SCHLIB_Blender:RES_10KR_1/20W_1%_R0201; Manufacturer (none) -> Stackpole Electronics Inc; PCB CHECk (none) -> PCB (N/A); Part Number RMCF0201FT10K0 -> (none); Part Number (Manufacturer) (none) -> RMCF0201FT10K0; Part Number (Vendor) (none) -> RMCF0201FT10K0TR-ND; SCH CHECK CHECKED -> SCH (N/A); Vendor (none) -> Digikey
- R1006: value 100R_1/20W -> 100R_1/20W_1%; symbol _SCHLIB_Blender:RES_100R_1/20W-R0201 -> _SCHLIB_Blender:RES_100R_1/20W_1%_R0201; Manufacturer (none) -> Stackpole Electronics Inc; PCB CHECk (none) -> PCB (N/A); Part Number RMCF0201FT100R -> (none); Part Number (Manufacturer) (none) -> RMCF0201FT100R; Part Number (Vendor) (none) -> RMCF0201FT100RTR-ND; SCH CHECK CHECKED -> SCH (N/A); Vendor (none) -> Digikey
- RV1001, RV1002: value PTC_500mA -> 0.5A_6V_0.15R; symbol _SCHLIB_Blender:PTC_PTS08056V050_F0805 -> _SCHLIB_Blender:FUSE_PTC_PTS08056V050_0.5A_1A_6V_F0805; Manufacturer (none) -> Eaton - Electronics Division; PCB CHECk (none) -> PCB (N/A); Part Number PTS08056V050 -> (none); Part Number (Manufacturer) (none) -> PTS08056V050; Part Number (Vendor) (none) -> 283-PTS08056V050TR-ND; SCH CHECK * -> SCH (N/A); Vendor (none) -> Digikey
- U1001: symbol _SCHLIB_Blender:PMIC_TPS613222ADBVR -> _SCHLIB_Blender:IC_PMIC_TPS613222ADBVR_SMPS-BOOST_5V_2.5A_SOT-753; Manufacturer (none) -> Texas Instruments; PCB CHECk (none) -> PCB (N/A); Package (none) -> SOT-753; Part Number TPS613222ADBVR -> (none); Part Number (Manufacturer) (none) -> TPS613222ADBVR; Part Number (Vendor) (none) -> 296-50503-2-ND; SCH CHECK * -> SCH (N/A); Vendor (none) -> Digikey
- U1002, U1004: symbol _SCHLIB_Blender:PMIC_TLV74033PDBVR -> _SCHLIB_Blender:IC_PMIC_TLV74033PDBVR_LDO_3.3V_0.3A_SOT-23-5; Manufacturer (none) -> Texas Instruments; PCB CHECk (none) -> PCB (N/A); Package (none) -> SOT-23-5; Part Number TLV74033PDBVR -> (none); Part Number (Manufacturer) (none) -> TLV74033PDBVR; Part Number (Vendor) (none) -> 296-TLV74033PDBVRTR-ND; SCH CHECK * -> SCH (N/A); Vendor (none) -> Digikey
- U1003: symbol _SCHLIB_Blender:PMIC_MCP73811T-420I/OT -> _SCHLIB_Blender:IC_PMIC_MCP73811T-420I/OT_CHARGER_1C_SOT-23-5; Manufacturer (none) -> Microchip Technology; PCB CHECk (none) -> PCB (N/A); Package (none) -> SOT-23-5; Part Number MCP73811T-420I/OT -> (none); Part Number (Manufacturer) (none) -> MCP73811T-420I/OT; Part Number (Vendor) (none) -> MCP73811T-420I/OTTR-ND; SCH CHECK * -> SCH (N/A); Vendor (none) -> Digikey
Other:
- moved on the sheet: C1001, C1002, C1003, C1004, C1005, C1006, C1008, C1010, D1001, D1002, D1003, F1001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
