File: Hardware/v1_20230918/Design Folder/_HW_Blender/[0501] - VIDEO SIG BUFF.kicad_sch (KiCad schematic)
At the start: 6 parts, among them U1201 MIC920YC5-TR

Commit message: Updating Library
Parts:
- C1201: symbol _SCHLIB_Blender:CAP_2u2F_6V3_X5R_C0201 -> _SCHLIB_Blender:CAP_CER_2u2F_6V3_X5R_C0201
- C1202: symbol _SCHLIB_Blender:CAP_100nF_6V3_X7R_C0201 -> _SCHLIB_Blender:CAP_CER_100nF_6V3_X7R_C0201
Changed lines of the file:
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@@
     )
   )
-  (symbol (lib_id "_SCHLIB_Blender:CAP_2u2F_6V3_X5R_C0201") (at 190.5 180.34 270) (unit 1)
+  (symbol (lib_id "_SCHLIB_Blender:CAP_CER_2u2F_6V3_X5R_C0201") (at 190.5 180.34 270) (unit 1)
     (in_bom yes) (on_board yes) (dnp no)
     (property "Reference" "C1201" (at 193.04 181.61 90)
@@
     )
   )
-  (symbol (lib_id "_SCHLIB_Blender:CAP_100nF_6V3_X7R_C0201") (at 212.09 180.34 270) (unit 1)
+  (symbol (lib_id "_SCHLIB_Blender:CAP_CER_100nF_6V3_X7R_C0201") (at 212.09 180.34 270) (unit 1)
     (in_bom yes) (on_board yes) (dnp no)
     (property "Reference" "C1202" (at 214.63 181.61 90)
@@
       (effects (font (size 1.27 1.27)) (justify left) hide)
     )
-    (property "SCH CHECK" "SCH (N/A)" (at 252.73 156.21 0)
+    (property "SCH CHECK" "SCH (N/A)" (at 252.73 158.75 0)
       (effects (font (size 1.27 1.27)) (justify left))
     )
@@
       (effects (font (size 1.27 1.27)) (justify left) hide)
     )
-    (property "Package" "SC-70-5" (at 252.73 158.75 0)
-      (effects (font (size 1.27 1.27)) (justify left))
-    )
+    (property "Package" "SC-70-5" (at 252.73 156.21 0)
+      (effects (font (size 1.27 1.27)) (justify left))
+    )
