File: Hardware/v1_20230918/Design Folder/_HW_Blender/[09] - OLED DRIVER.kicad_sch (KiCad schematic)
At the start: 6 parts, among them J901 RECEPT_6X1_VERT_2.54MM

Commit message: Updating Library
Parts:
- C901: symbol _SCHLIB_Blender:CAP_1uF_6V3_X5R_C0201 -> _SCHLIB_Blender:CAP_CER_1uF_6V3_X5R_C0201
Changed lines of the file:
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@@
     (effects (font (size 1.27 1.27)) (justify right))
   )
-  (symbol (lib_id "_SCHLIB_Blender:CAP_1uF_6V3_X5R_C0201") (at 264.16 180.34 270) (unit 1)
+  (symbol (lib_id "_SCHLIB_Blender:CAP_CER_1uF_6V3_X5R_C0201") (at 264.16 180.34 270) (unit 1)
     (in_bom yes) (on_board yes) (dnp no)
     (property "Reference" "C901" (at 266.7 181.61 90)
