File: Hardware/v1_20230918/Design Folder/_HW_Blender/[04] - TOSLINK RXTX.kicad_sch (KiCad schematic)
At the start: 12 parts, among them J401 PLR237/T10BK, J402 TOTX1350(F), U401 SN74LVC1G17DBVR, U402 SN74LVC1G17DBVR

Commit message: Updating Library
Parts:
- C401: symbol _SCHLIB_Blender:CAP_680pF_50V_X7R_C0402 -> _SCHLIB_Blender:CAP_CER_680pF_50V_X7R_C0402
- C402, C403, C404: symbol _SCHLIB_Blender:CAP_100nF_6V3_X7R_C0201 -> _SCHLIB_Blender:CAP_CER_100nF_6V3_X7R_C0201
Changed lines of the file:
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@@
       (effects (font (size 1.27 1.27)) (justify left) hide)
     )
-    (property "SCH CHECK" "SCH (N/A)" (at 204.47 160.02 0)
+    (property "SCH CHECK" "SCH (N/A)" (at 204.47 162.56 0)
       (effects (font (size 1.27 1.27)) (justify left))
     )
@@
       (effects (font (size 1.27 1.27)) (justify left) hide)
     )
-    (property "PCB CHECK" "PCB (N/A)" (at 204.47 162.56 0)
+    (property "PCB CHECK" "PCB (N/A)" (at 204.47 165.1 0)
       (effects (font (size 1.27 1.27)) (justify left))
     )
@@
       (effects (font (size 1.27 1.27)) (justify left) hide)
     )
-    (property "Package" "SOT23-5" (at 204.47 165.1 0)
+    (property "Package" "SOT23-5" (at 204.47 160.02 0)
       (effects (font (size 1.27 1.27)) (justify left))
     )
@@
     )
   )
-  (symbol (lib_id "_SCHLIB_Blender:CAP_100nF_6V3_X7R_C0201") (at 266.7 176.53 270) (unit 1)
+  (symbol (lib_id "_SCHLIB_Blender:CAP_CER_100nF_6V3_X7R_C0201") (at 266.7 176.53 270) (unit 1)
     (in_bom yes) (on_board yes) (dnp no)
     (property "Reference" "C404" (at 269.24 177.8 90)
@@
     )
   )
-  (symbol (lib_id "_SCHLIB_Blender:CAP_100nF_6V3_X7R_C0201") (at 176.53 176.53 270) (unit 1)
+  (symbol (lib_id "_SCHLIB_Blender:CAP_CER_100nF_6V3_X7R_C0201") (at 176.53 176.53 270) (unit 1)
     (in_bom yes) (on_board yes) (dnp no)
     (property "Reference" "C403" (at 179.07 177.8 90)
@@
       (effects (font (size 1.27 1.27)) (justify left) hide)
     )
-    (property "SCH CHECK" "SCH (N/A)" (at 295.91 160.02 0)
+    (property "SCH CHECK" "SCH (N/A)" (at 295.91 162.56 0)
       (effects (font (size 1.27 1.27)) (justify left))
     )
@@
       (effects (font (size 1.27 1.27)) (justify left) hide)
     )
-    (property "PCB CHECK" "PCB (N/A)" (at 295.91 162.56 0)
+    (property "PCB CHECK" "PCB (N/A)" (at 295.91 165.1 0)
       (effects (font (size 1.27 1.27)) (justify left))
     )
@@
       (effects (font (size 1.27 1.27)) (justify left) hide)
     )
-    (property "Package" "SOT23-5" (at 295.91 165.1 0)
+    (property "Package" "SOT23-5" (at 295.91 160.02 0)
       (effects (font (size 1.27 1.27)) (justify left))
     )
@@
     )
   )
-  (symbol (lib_id "_SCHLIB_Blender:CAP_680pF_50V_X7R_C0402") (at 337.82 160.02 0) (unit 1)
+  (symbol (lib_id "_SCHLIB_Blender:CAP_CER_680pF_50V_X7R_C0402") (at 337.82 160.02 0) (unit 1)
     (in_bom yes) (on_board yes) (dnp no)
     (property "Reference" "C401" (at 353.06 158.75 0)
@@
     )
   )
-  (symbol (lib_id "_SCHLIB_Blender:CAP_100nF_6V3_X7R_C0201") (at 66.04 171.45 270) (unit 1)
+  (symbol (lib_id "_SCHLIB_Blender:CAP_CER_100nF_6V3_X7R_C0201") (at 66.04 171.45 270) (unit 1)
     (in_bom yes) (on_board yes) (dnp no)
     (property "Reference" "C402" (at 68.58 172.72 90)
@@
       (effects (font (size 1.27 1.27)) (justify left) hide)
     )
-    (property "SCH CHECK" "SCH (N/A)" (at 452.12 160.02 0)
+    (property "SCH CHECK" "SCH (N/A)" (at 452.12 162.56 0)
       (effects (font (size 1.27 1.27)) (justify left))
     )
@@
       (effects (font (size 1.27 1.27)) (justify left) hide)
     )
-    (property "Package" "THD-RA" (at 452.12 162.56 0)
-      (effects (font (size 1.27 1.27)) (justify left))
-    )
+    (property "Package" "THD-RA" (at 452.12 160.02 0)
+      (effects (font (size 1.27 1.27)) (justify left))
+    )
