File: Hardware/v1_20230918/Design Folder/_HW_Blender/[05] - BUFFERED VGA INPUT.kicad_sch (KiCad schematic)
At the start: 21 parts, among them J501 DSUB_15POS_MALE_RA, U501 SN74LVC1G17DBVR, U502 SN74LVC1G17DBVR

Commit message: Updating Library
Parts:
- C501, C503: symbol _SCHLIB_Blender:CAP_2u2F_6V3_X5R_C0201 -> _SCHLIB_Blender:CAP_CER_2u2F_6V3_X5R_C0201
- C502, C504: symbol _SCHLIB_Blender:CAP_100nF_6V3_X7R_C0201 -> _SCHLIB_Blender:CAP_CER_100nF_6V3_X7R_C0201
Changed lines of the file:
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@@
     )
   )
-  (symbol (lib_id "_SCHLIB_Blender:CAP_2u2F_6V3_X5R_C0201") (at 306.07 247.65 270) (unit 1)
+  (symbol (lib_id "_SCHLIB_Blender:CAP_CER_2u2F_6V3_X5R_C0201") (at 306.07 247.65 270) (unit 1)
     (in_bom yes) (on_board yes) (dnp no)
     (property "Reference" "C503" (at 308.61 248.92 90)
@@
       (effects (font (size 1.27 1.27)) (justify left) hide)
     )
-    (property "SCH CHECK" "SCH (N/A)" (at 354.33 187.96 0)
+    (property "SCH CHECK" "SCH (N/A)" (at 354.33 190.5 0)
       (effects (font (size 1.27 1.27)) (justify left))
     )
@@
       (effects (font (size 1.27 1.27)) (justify left) hide)
     )
-    (property "PCB CHECK" "PCB (N/A)" (at 354.33 190.5 0)
+    (property "PCB CHECK" "PCB (N/A)" (at 354.33 193.04 0)
       (effects (font (size 1.27 1.27)) (justify left))
     )
@@
       (effects (font (size 1.27 1.27)) (justify left) hide)
     )
-    (property "Package" "SOT23-5" (at 354.33 193.04 0)
+    (property "Package" "SOT23-5" (at 354.33 187.96 0)
       (effects (font (size 1.27 1.27)) (justify left))
     )
@@
       (effects (font (size 1.27 1.27)) (justify left) hide)
     )
-    (property "SCH CHECK" "SCH (N/A)" (at 354.33 228.6 0)
+    (property "SCH CHECK" "SCH (N/A)" (at 354.33 231.14 0)
       (effects (font (size 1.27 1.27)) (justify left))
     )
@@
       (effects (font (size 1.27 1.27)) (justify left) hide)
     )
-    (property "PCB CHECK" "PCB (N/A)" (at 354.33 231.14 0)
+    (property "PCB CHECK" "PCB (N/A)" (at 354.33 233.68 0)
       (effects (font (size 1.27 1.27)) (justify left))
     )
@@
       (effects (font (size 1.27 1.27)) (justify left) hide)
     )
-    (property "Package" "SOT23-5" (at 354.33 233.68 0)
+    (property "Package" "SOT23-5" (at 354.33 228.6 0)
       (effects (font (size 1.27 1.27)) (justify left))
     )
@@
     )
   )
-  (symbol (lib_id "_SCHLIB_Blender:CAP_2u2F_6V3_X5R_C0201") (at 306.07 207.01 270) (unit 1)
+  (symbol (lib_id "_SCHLIB_Blender:CAP_CER_2u2F_6V3_X5R_C0201") (at 306.07 207.01 270) (unit 1)
     (in_bom yes) (on_board yes) (dnp no)
     (property "Reference" "C501" (at 308.61 208.28 90)
@@
     )
   )
-  (symbol (lib_id "_SCHLIB_Blender:CAP_100nF_6V3_X7R_C0201") (at 328.93 207.01 270) (unit 1)
+  (symbol (lib_id "_SCHLIB_Blender:CAP_CER_100nF_6V3_X7R_C0201") (at 328.93 207.01 270) (unit 1)
     (in_bom yes) (on_board yes) (dnp no)
     (property "Reference" "C502" (at 331.47 208.28 90)
@@
       (effects (font (size 1.27 1.27)) (justify left) hide)
     )
-    (property "SCH CHECK" "SCH (N/A)" (at 140.97 165.1 0)
+    (property "SCH CHECK" "SCH (N/A)" (at 140.97 167.64 0)
       (effects (font (size 1.27 1.27)) (justify left))
     )
@@
       (effects (font (size 1.27 1.27)) (justify left) hide)
     )
-    (property "Package" "THD-R/A" (at 140.97 167.64 0)
+    (property "Package" "THD-R/A" (at 140.97 165.1 0)
       (effects (font (size 1.27 1.27)) (justify left))
     )
@@
     )
   )
-  (symbol (lib_id "_SCHLIB_Blender:CAP_100nF_6V3_X7R_C0201") (at 328.93 247.65 270) (unit 1)
+  (symbol (lib_id "_SCHLIB_Blender:CAP_CER_100nF_6V3_X7R_C0201") (at 328.93 247.65 270) (unit 1)
     (in_bom yes) (on_board yes) (dnp no)
     (property "Reference" "C504" (at 331.47 248.92 90)
