File: Hardware/v1_20230918/Design Folder/_HW_Blender/[06] - ISOLATED WS28xx DRIVER.kicad_sch (KiCad schematic)
At the start: 41 parts, among them J601 MHDR_2X1_VERT_1.27MM, J602 RECEPT_4X1_VERT_1.27MM, U601 SN74LVC1G17DBVR, U602 ISO7720FDR, U603 SN74LVC1G17DBVR, U604 DLPT05A-7, U605 DLPT05A-7

Commit message: Updating Library
Parts:
- C601, C602, C603, C604, C605, C606, C607, C608, C609, C611: symbol _SCHLIB_Blender:CAP_2u2F_6V3_X5R_C0201 -> _SCHLIB_Blender:CAP_CER_2u2F_6V3_X5R_C0201
- C610: symbol _SCHLIB_Blender:CAP_10uF_16V_X5R_C0603 -> _SCHLIB_Blender:CAP_CER_10uF_16V_X5R_C0603
- U602: Package 8-SOIC (0.154", 3.90mm Width) -> 8-SOIC (3.90mm Width)
Changed lines of the file:
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@@
     )
   )
-  (symbol (lib_id "_SCHLIB_Blender:CAP_2u2F_6V3_X5R_C0201") (at 195.58 285.75 270) (unit 1)
+  (symbol (lib_id "_SCHLIB_Blender:CAP_CER_2u2F_6V3_X5R_C0201") (at 195.58 285.75 270) (unit 1)
     (in_bom yes) (on_board yes) (dnp no)
     (property "Reference" "C609" (at 198.12 287.02 90)
@@
     )
   )
-  (symbol (lib_id "_SCHLIB_Blender:CAP_2u2F_6V3_X5R_C0201") (at 146.05 208.28 270) (unit 1)
+  (symbol (lib_id "_SCHLIB_Blender:CAP_CER_2u2F_6V3_X5R_C0201") (at 146.05 208.28 270) (unit 1)
     (in_bom yes) (on_board yes) (dnp no)
     (property "Reference" "C605" (at 148.59 209.55 90)
@@
     )
   )
-  (symbol (lib_id "_SCHLIB_Blender:CAP_2u2F_6V3_X5R_C0201") (at 129.54 336.55 270) (unit 1)
+  (symbol (lib_id "_SCHLIB_Blender:CAP_CER_2u2F_6V3_X5R_C0201") (at 129.54 336.55 270) (unit 1)
     (in_bom yes) (on_board yes) (dnp no)
     (property "Reference" "C611" (at 132.08 337.82 90)
@@
       (effects (font (size 1.27 1.27)) (justify left) hide)
     )
-    (property "SCH CHECK" "SCH (N/A)" (at 228.6 298.45 0)
+    (property "SCH CHECK" "SCH (N/A)" (at 228.6 300.99 0)
       (effects (font (size 1.27 1.27)) (justify left))
     )
@@
       (effects (font (size 1.27 1.27)) (justify left) hide)
     )
-    (property "Package" "8-SOIC (0.154\", 3.90mm Width)" (at 228.6 300.99 0)
+    (property "Package" "8-SOIC (3.90mm Width)" (at 228.6 298.45 0)
       (effects (font (size 1.27 1.27)) (justify left))
     )
@@
     )
   )
-  (symbol (lib_id "_SCHLIB_Blender:CAP_2u2F_6V3_X5R_C0201") (at 219.71 137.16 270) (unit 1)
+  (symbol (lib_id "_SCHLIB_Blender:CAP_CER_2u2F_6V3_X5R_C0201") (at 219.71 137.16 270) (unit 1)
     (in_bom yes) (on_board yes) (dnp no)
     (property "Reference" "C601" (at 222.25 138.43 90)
@@
     )
   )
-  (symbol (lib_id "_SCHLIB_Blender:CAP_2u2F_6V3_X5R_C0201") (at 144.78 134.62 270) (unit 1)
+  (symbol (lib_id "_SCHLIB_Blender:CAP_CER_2u2F_6V3_X5R_C0201") (at 144.78 134.62 270) (unit 1)
     (in_bom yes) (on_board yes) (dnp no)
     (property "Reference" "C604" (at 147.32 135.89 90)
@@
     )
   )
-  (symbol (lib_id "_SCHLIB_Blender:CAP_2u2F_6V3_X5R_C0201") (at 220.98 208.28 270) (unit 1)
+  (symbol (lib_id "_SCHLIB_Blender:CAP_CER_2u2F_6V3_X5R_C0201") (at 220.98 208.28 270) (unit 1)
     (in_bom yes) (on_board yes) (dnp no)
     (property "Reference" "C606" (at 223.52 209.55 90)
@@
     )
   )
-  (symbol (lib_id "_SCHLIB_Blender:CAP_2u2F_6V3_X5R_C0201") (at 299.72 137.16 270) (unit 1)
+  (symbol (lib_id "_SCHLIB_Blender:CAP_CER_2u2F_6V3_X5R_C0201") (at 299.72 137.16 270) (unit 1)
     (in_bom yes) (on_board yes) (dnp no)
     (property "Reference" "C602" (at 302.26 138.43 90)
@@
     )
   )
-  (symbol (lib_id "_SCHLIB_Blender:CAP_10uF_16V_X5R_C0603") (at 266.7 285.75 270) (unit 1)
+  (symbol (lib_id "_SCHLIB_Blender:CAP_CER_10uF_16V_X5R_C0603") (at 266.7 285.75 270) (unit 1)
     (in_bom yes) (on_board yes) (dnp no)
     (property "Reference" "C610" (at 269.24 287.02 90)
@@
     )
   )
-  (symbol (lib_id "_SCHLIB_Blender:CAP_2u2F_6V3_X5R_C0201") (at 388.62 137.16 270) (unit 1)
+  (symbol (lib_id "_SCHLIB_Blender:CAP_CER_2u2F_6V3_X5R_C0201") (at 388.62 137.16 270) (unit 1)
     (in_bom yes) (on_board yes) (dnp no)
     (property "Reference" "C603" (at 391.16 138.43 90)
@@
     )
   )
-  (symbol (lib_id "_SCHLIB_Blender:CAP_2u2F_6V3_X5R_C0201") (at 298.45 208.28 270) (unit 1)
+  (symbol (lib_id "_SCHLIB_Blender:CAP_CER_2u2F_6V3_X5R_C0201") (at 298.45 208.28 270) (unit 1)
     (in_bom yes) (on_board yes) (dnp no)
     (property "Reference" "C607" (at 300.99 209.55 90)
@@
     )
   )
-  (symbol (lib_id "_SCHLIB_Blender:CAP_2u2F_6V3_X5R_C0201") (at 379.73 208.28 270) (unit 1)
+  (symbol (lib_id "_SCHLIB_Blender:CAP_CER_2u2F_6V3_X5R_C0201") (at 379.73 208.28 270) (unit 1)
     (in_bom yes) (on_board yes) (dnp no)
     (property "Reference" "C608" (at 382.27 209.55 90)
