File: Hardware/v1_20230918/Design Folder/_HW_Blender/[07] - ISOLATED DMX.kicad_sch (KiCad schematic)
At the start: 22 parts, among them J701 RECEPT_3X1_VERT_1.27MM, U701 1S4E_0505S1.5U, U702 SN74LVC1G17DBVR, U703 CDSOT23-SM712, U704 MAX22028AWA+, U705 SN74LVC1G17DBVR

Commit message: Updating Library
Parts:
- C701, C702, C703, C704, C705, C706: symbol _SCHLIB_Blender:CAP_10uF_16V_X5R_C0603 -> _SCHLIB_Blender:CAP_CER_10uF_16V_X5R_C0603
- U704: Package 8-SOIC (0.209", 5.30mm Width) -> 8-SOIC (5.30mm Width)
Changed lines of the file:
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@@
     )
   )
-  (symbol (lib_id "_SCHLIB_Blender:CAP_10uF_16V_X5R_C0603") (at 147.32 184.15 90) (mirror x) (unit 1)
+  (symbol (lib_id "_SCHLIB_Blender:CAP_CER_10uF_16V_X5R_C0603") (at 147.32 184.15 90) (mirror x) (unit 1)
     (in_bom yes) (on_board yes) (dnp no)
     (property "Reference" "C703" (at 149.86 185.42 90)
@@
     )
   )
-  (symbol (lib_id "_SCHLIB_Blender:CAP_10uF_16V_X5R_C0603") (at 220.98 222.25 270) (unit 1)
+  (symbol (lib_id "_SCHLIB_Blender:CAP_CER_10uF_16V_X5R_C0603") (at 220.98 222.25 270) (unit 1)
     (in_bom yes) (on_board yes) (dnp no)
     (property "Reference" "C705" (at 223.52 223.52 90)
@@
     )
   )
-  (symbol (lib_id "_SCHLIB_Blender:CAP_10uF_16V_X5R_C0603") (at 218.44 134.62 270) (unit 1)
+  (symbol (lib_id "_SCHLIB_Blender:CAP_CER_10uF_16V_X5R_C0603") (at 218.44 134.62 270) (unit 1)
     (in_bom yes) (on_board yes) (dnp no)
     (property "Reference" "C701" (at 220.98 135.89 90)
@@
       (effects (font (size 1.27 1.27)) (justify left) hide)
     )
-    (property "SCH CHECK" "SCH (N/A)" (at 246.38 205.74 0)
+    (property "SCH CHECK" "SCH (N/A)" (at 246.38 208.28 0)
       (effects (font (size 1.27 1.27)) (justify left))
     )
@@
       (effects (font (size 1.27 1.27)) (justify left) hide)
     )
-    (property "Package" "8-SOIC (0.209\", 5.30mm Width)" (at 246.38 208.28 0)
+    (property "Package" "8-SOIC (5.30mm Width)" (at 246.38 205.74 0)
       (effects (font (size 1.27 1.27)) (justify left))
     )
@@
     )
   )
-  (symbol (lib_id "_SCHLIB_Blender:CAP_10uF_16V_X5R_C0603") (at 280.67 134.62 270) (unit 1)
+  (symbol (lib_id "_SCHLIB_Blender:CAP_CER_10uF_16V_X5R_C0603") (at 280.67 134.62 270) (unit 1)
     (in_bom yes) (on_board yes) (dnp no)
     (property "Reference" "C702" (at 283.21 135.89 90)
@@
     )
   )
-  (symbol (lib_id "_SCHLIB_Blender:CAP_10uF_16V_X5R_C0603") (at 85.09 224.79 270) (unit 1)
+  (symbol (lib_id "_SCHLIB_Blender:CAP_CER_10uF_16V_X5R_C0603") (at 85.09 224.79 270) (unit 1)
     (in_bom yes) (on_board yes) (dnp no)
     (property "Reference" "C706" (at 87.63 226.06 90)
@@
     )
   )
-  (symbol (lib_id "_SCHLIB_Blender:CAP_10uF_16V_X5R_C0603") (at 283.21 176.53 270) (unit 1)
+  (symbol (lib_id "_SCHLIB_Blender:CAP_CER_10uF_16V_X5R_C0603") (at 283.21 176.53 270) (unit 1)
     (in_bom yes) (on_board yes) (dnp no)
     (property "Reference" "C704" (at 285.75 177.8 90)
