File: Hardware/v1_20230918/Design Folder/_HW_Blender/[10] - Power Supply.kicad_sch (KiCad schematic)
At the start: 36 parts, among them J1001 MHDR_2X1_VERT_1.27MM, J1002 MICRO B USB_RA, Q1001 SI4455DY-T1-GE3, Q1002 RN1130MFV,L3F, U1001 TPS613222ADBVR, U1002 TLV74033PDBVR, U1003 MCP73811T-420I/OT, U1004 TLV74033PDBVR

Commit message: Updating Library
Parts:
- C1001: symbol _SCHLIB_Blender:CAP_680pF_50V_X7R_C0402 -> _SCHLIB_Blender:CAP_CER_680pF_50V_X7R_C0402
- C1002, C1003, C1004, C1007, C1008, C1009, C1010: symbol _SCHLIB_Blender:CAP_10uF_16V_X5R_C0603 -> _SCHLIB_Blender:CAP_CER_10uF_16V_X5R_C0603
- C1005, C1006: symbol _SCHLIB_Blender:CAP_1uF_6V3_X5R_C0201 -> _SCHLIB_Blender:CAP_CER_1uF_6V3_X5R_C0201
Changed lines of the file:
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@@
     )
   )
-  (symbol (lib_id "_SCHLIB_Blender:CAP_680pF_50V_X7R_C0402") (at 306.07 120.65 180) (unit 1)
+  (symbol (lib_id "_SCHLIB_Blender:CAP_CER_680pF_50V_X7R_C0402") (at 306.07 120.65 180) (unit 1)
     (in_bom yes) (on_board yes) (dnp no)
     (property "Reference" "C1001" (at 308.61 119.38 0)
@@
     )
   )
-  (symbol (lib_id "_SCHLIB_Blender:CAP_1uF_6V3_X5R_C0201") (at 389.89 237.49 270) (unit 1)
+  (symbol (lib_id "_SCHLIB_Blender:CAP_CER_1uF_6V3_X5R_C0201") (at 389.89 237.49 270) (unit 1)
     (in_bom yes) (on_board yes) (dnp no)
     (property "Reference" "C1005" (at 392.43 238.76 90)
@@
     )
   )
-  (symbol (lib_id "_SCHLIB_Blender:CAP_10uF_16V_X5R_C0603") (at 91.44 228.6 270) (unit 1)
+  (symbol (lib_id "_SCHLIB_Blender:CAP_CER_10uF_16V_X5R_C0603") (at 91.44 228.6 270) (unit 1)
     (in_bom yes) (on_board yes) (dnp no)
     (property "Reference" "C1007" (at 93.98 229.87 90)
@@
     )
   )
-  (symbol (lib_id "_SCHLIB_Blender:CAP_10uF_16V_X5R_C0603") (at 393.7 171.45 270) (unit 1)
+  (symbol (lib_id "_SCHLIB_Blender:CAP_CER_10uF_16V_X5R_C0603") (at 393.7 171.45 270) (unit 1)
     (in_bom yes) (on_board yes) (dnp no)
     (property "Reference" "C1004" (at 396.24 172.72 90)
@@
     )
   )
-  (symbol (lib_id "_SCHLIB_Blender:CAP_10uF_16V_X5R_C0603") (at 317.5 170.18 270) (unit 1)
+  (symbol (lib_id "_SCHLIB_Blender:CAP_CER_10uF_16V_X5R_C0603") (at 317.5 170.18 270) (unit 1)
     (in_bom yes) (on_board yes) (dnp no)
     (property "Reference" "C1003" (at 320.04 171.45 90)
@@
     )
   )
-  (symbol (lib_id "_SCHLIB_Blender:CAP_1uF_6V3_X5R_C0201") (at 439.42 237.49 270) (unit 1)
+  (symbol (lib_id "_SCHLIB_Blender:CAP_CER_1uF_6V3_X5R_C0201") (at 439.42 237.49 270) (unit 1)
     (in_bom yes) (on_board yes) (dnp no)
     (property "Reference" "C1006" (at 441.96 238.76 90)
@@
     )
   )
-  (symbol (lib_id "_SCHLIB_Blender:CAP_10uF_16V_X5R_C0603") (at 205.74 236.22 270) (unit 1)
+  (symbol (lib_id "_SCHLIB_Blender:CAP_CER_10uF_16V_X5R_C0603") (at 205.74 236.22 270) (unit 1)
     (in_bom yes) (on_board yes) (dnp no)
     (property "Reference" "C1008" (at 208.28 237.49 90)
@@
     )
   )
-  (symbol (lib_id "_SCHLIB_Blender:CAP_10uF_16V_X5R_C0603") (at 205.74 288.29 270) (unit 1)
+  (symbol (lib_id "_SCHLIB_Blender:CAP_CER_10uF_16V_X5R_C0603") (at 205.74 288.29 270) (unit 1)
     (in_bom yes) (on_board yes) (dnp no)
     (property "Reference" "C1010" (at 208.28 289.56 90)
@@
     )
   )
-  (symbol (lib_id "_SCHLIB_Blender:CAP_10uF_16V_X5R_C0603") (at 204.47 170.18 270) (unit 1)
+  (symbol (lib_id "_SCHLIB_Blender:CAP_CER_10uF_16V_X5R_C0603") (at 204.47 170.18 270) (unit 1)
     (in_bom yes) (on_board yes) (dnp no)
     (property "Reference" "C1002" (at 207.01 171.45 90)
@@
     )
   )
-  (symbol (lib_id "_SCHLIB_Blender:CAP_10uF_16V_X5R_C0603") (at 91.44 283.21 270) (unit 1)
+  (symbol (lib_id "_SCHLIB_Blender:CAP_CER_10uF_16V_X5R_C0603") (at 91.44 283.21 270) (unit 1)
     (in_bom yes) (on_board yes) (dnp no)
     (property "Reference" "C1009" (at 93.98 284.48 90)

Commit message: Updating 3D components
Parts:
- J1002: footprint Connector_USB:USB_Micro-B_Amphenol_10118194_Horizontal -> _PCBLIB_Blender:USB_Micro-B_Amphenol_10118194_Horizontal
Changed lines of the file:
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@@
       (effects (font (size 1.27 1.27)) (justify left))
     )
-    (property "Footprint" "Connector_USB:USB_Micro-B_Amphenol_10118194_Horizontal" (at 302.26 217.17 0)
+    (property "Footprint" "_PCBLIB_Blender:USB_Micro-B_Amphenol_10118194_Horizontal" (at 302.26 217.17 0)
       (effects (font (size 1.27 1.27)) (justify left) hide)
     )
@@
       (effects (font (size 1.27 1.27)) (justify left))
     )
-    (property "Part Number (Manufacturer)" "10118194-0001LF" (at 302.26 214.63 0)
+    (property "Part Number (Manufacturer)" "10118194-0001LF" (at 302.26 212.09 0)
       (effects (font (size 1.27 1.27)) (justify left) hide)
     )
@@
       (effects (font (size 1.27 1.27)) (justify left))
     )
-    (property "Manufacturer" "Amphenol ICC (FCI)" (at 299.72 232.41 0)
+    (property "Manufacturer" "Amphenol ICC (FCI)" (at 302.26 209.55 0)
       (effects (font (size 1.27 1.27)) (justify left) hide)
     )
-    (property "Part Number (Vendor)" "609-4618-2-ND" (at 299.72 232.41 0)
+    (property "Part Number (Vendor)" "609-4618-2-ND" (at 302.26 214.63 0)
       (effects (font (size 1.27 1.27)) (justify left) hide)
     )
-    (property "Vendor" "Digikey" (at 299.72 232.41 0)
+    (property "Vendor" "Digikey" (at 302.26 207.01 0)
       (effects (font (size 1.27 1.27)) (justify left) hide)
     )
