File: Hardware/v1_20230918/Design Folder/_HW_Blender/_HW_Blender.kicad_pcb (KiCad board)
At the start: 4 copper layers, 49.7 x 49.7 mm, 217 parts, among them J1001 MHDR_2X1_VERT_1.27MM, J1002 MICRO B USB_RA, J301 RECEPT_4X1_VERT_1.27MM, J401 PLR237/T10BK, J402 TOTX1350(F), J501 DSUB_15POS_MALE_RA, J601 MHDR_2X1_VERT_1.27MM, J602 RECEPT_4X1_VERT_1.27MM, J701 RECEPT_3X1_VERT_1.27MM, J801 MHDR_2X1_VERT_1.27MM, J802 MHDR_2X1_VERT_1.27MM, J901 RECEPT_6X1_VERT_2.54MM, Q1001 SI4455DY-T1-GE3, Q1002 RN1130MFV,L3F, U1001 TPS613222ADBVR, U1002 TLV74033PDBVR, U1003 MCP73811T-420I/OT, U1004 TLV74033PDBVR, U1201 MIC920YC5-TR, U1301 MIC920YC5-TR, U1401 MIC920YC5-TR, U301 STM32F446RCT6TR, U401 SN74LVC1G17DBVR, U402 SN74LVC1G17DBVR, U501 SN74LVC1G17DBVR, U502 SN74LVC1G17DBVR, U601 SN74LVC1G17DBVR, U602 ISO7720FDR, U603 SN74LVC1G17DBVR, U604 DLPT05A-7, U605 DLPT05A-7, U701 1S4E_0505S1.5U, U702 SN74LVC1G17DBVR, U703 CDSOT23-SM712, U704 MAX22028AWA+, U705 SN74LVC1G17DBVR, U801 PAM8003DR, U802 PCM1754DBQR, X301 16MHz_12pF_10ppm

Commit message: Updating 3D components
Parts:
- J1002: footprint Connector_USB:USB_Micro-B_Amphenol_10118194_Horizontal -> _PCBLIB_Blender:USB_Micro-B_Amphenol_10118194_Horizontal
- U801: footprint Package_SO:SOP-16_3.9x9.9mm_P1.27mm -> _PCBLIB_Blender:SOP-16_3.9x9.9mm_P1.27mm
